Commit message: Added fenders

File: jackal_description/urdf/jackal.urdf.xacro (robot description, xacro)
@@ -113,5 +113,5 @@
       </inertial>
   </link>
-  <xacro:unless value="$(optenv JACKAL_FRONT_ACCESSORY_FENDER 0)">
+  <!-- <xacro:unless value="$(optenv JACKAL_FRONT_ACCESSORY_FENDER 0)">
     <link name="front_fender_link">
       <visual>
@@ -143,6 +143,6 @@
     <parent link="chassis_link" />
     <child link="front_fender_link" />
-  </joint>
-  <xacro:unless value="$(optenv JACKAL_REAR_ACCESSORY_FENDER 0)">
+  </joint> -->
+  <!-- <xacro:unless value="$(optenv JACKAL_REAR_ACCESSORY_FENDER 0)">
     <link name="rear_fender_link">
       <visual>
@@ -174,5 +174,5 @@
     <parent link="chassis_link" />
     <child link="rear_fender_link" />
-  </joint>
+  </joint> -->
   <!-- TODO: Make this internal_imu_link or something, and use a mixed-in xacro
        to supply the joint between it and imu_link. This is important so that imu_link

Commit message: Removed fenders and extras Added fender mounts

File: jackal_description/urdf/jackal.urdf.xacro (robot description, xacro)
@@ -113,66 +113,4 @@
       </inertial>
   </link>
-  <!-- <xacro:unless value="$(optenv JACKAL_FRONT_ACCESSORY_FENDER 0)">
-    <link name="front_fender_link">
-      <visual>
-        <geometry>
-          <mesh filename="package://jackal_description/meshes/jackal-fender.stl"/>
-        </geometry>
-        <material name="yellow" />
-      </visual>
-    </link>
-  </xacro:unless>
-  <xacro:if value="$(optenv JACKAL_FRONT_ACCESSORY_FENDER 0)">
-    <link name="front_fender_link">
-      <visual>
-        <geometry>
-          <mesh filename="package://jackal_description/meshes/accessory_fender.stl"/>
-        </geometry>
-        <material name="yellow" />
-      </visual>
-    </link>
-    <link name="front_fender_accessory_link"/>
-    <joint name="front_fender_accessory_joint" type="fixed">
-      <origin xyz="0.25629 0 0.07455" rpy="${PI} 0 0" />
-      <parent link="front_fender_link" />
-      <child link="front_fender_accessory_link" />
-    </joint>
-  </xacro:if>
-  <joint name="front_fender_joint" type="fixed">
-    <origin xyz="0 0 0" rpy="0 0 0"/>
-    <parent link="chassis_link" />
-    <child link="front_fender_link" />
-  </joint> -->
-  <!-- <xacro:unless value="$(optenv JACKAL_REAR_ACCESSORY_FENDER 0)">
-    <link name="rear_fender_link">
-      <visual>
-        <geometry>
-          <mesh filename="package://jackal_description/meshes/jackal-fender.stl"/>
-        </geometry>
-        <material name="yellow" />
-      </visual>
-    </link>
-  </xacro:unless>
-  <xacro:if value="$(optenv JACKAL_REAR_ACCESSORY_FENDER 0)">
-    <link name="rear_fender_link">
-      <visual>
-        <geometry>
-          <mesh filename="package://jackal_description/meshes/accessory_fender.stl"/>
-        </geometry>
-        <material name="yellow" />
-      </visual>
-    </link>
-    <link name="rear_fender_accessory_link"/>
-    <joint name="rear_fender_accessory_joint" type="fixed">
-      <origin xyz="0.25629 0 0.07455" rpy="${PI} 0 0" />
-      <parent link="rear_fender_link" />
-      <child link="rear_fender_accessory_link" />
-    </joint>
-  </xacro:if>
-  <joint name="rear_fender_joint" type="fixed">
-    <origin xyz="0 0 0" rpy="0 0 ${PI}"/>
-    <parent link="chassis_link" />
-    <child link="rear_fender_link" />
-  </joint> -->
   <!-- TODO: Make this internal_imu_link or something, and use a mixed-in xacro
        to supply the joint between it and imu_link. This is important so that imu_link
@@ -223,4 +161,16 @@
     <origin xyz="${mount_spacing} 0 0" />
   </joint>
+  <link name="front_fender_mount"></link>
+  <joint name="front_fender_mount_joint" type="fixed">
+    <parent link="chassis_link" />
+    <child link="front_fender_mount" />
+    <origin xyz="0 0 0" />
+  </joint>
+  <link name="rear_fender_mount"></link>
+  <joint name="rear_fender_mount_joint" type="fixed">
+    <parent link="chassis_link" />
+    <child link="rear_fender_mount" />
+    <origin xyz="0 0 0" rpy="0 0 ${PI}"/>
+  </joint>
   <ros2_control name="jackal_hardware" type="system">
     <hardware>
@@ -260,5 +210,3 @@
        default each one to off.-->
   <xacro:include filename="$(arg accessories)" />
-  <!-- Optional custom includes. -->
-  <xacro:include filename="$(optenv JACKAL_URDF_EXTRAS empty.urdf)" />
 </robot>
